File: hardware/pcb-design.kicad_pcb (KiCad board)
At the start: 2 copper layers, 137 parts, among them SW62 RotaryEncoder_Switch

Commit message: Routing done
Parts:
- removed A1: RaspberryPi_Pico, Module:RaspberryPi_Pico_Common_Unspecified
- removed SW62: RotaryEncoder_Switch, Rotary_Encoder:RotaryEncoder_Alps_EC11E-Switch_Vertical_H20mm
- added U1: RP2040-Matrix, PCM_marbastlib-xp-promicroish:RP2040-Matrix_AC, F.Cu at (173.5, -134.3)
- moved D14 82.8 mm to (153.8, -127.1)
- moved D61 82.8 mm to (145.1, -51.5)
- moved D62 82.8 mm to (164.1, -71.0)
- moved D63 82.8 mm to (183.1, -70.5)
- moved D65 82.8 mm to (183.0, -52.5)
- moved MX14 82.8 mm to (134.9, -133.3)
- moved D11 82.8 mm to (77.8, -127.0)
- moved D12 82.8 mm to (96.8, -127.3)
- moved D15 82.8 mm to (-103.1, -110.0)
- moved D16 82.8 mm to (-83.9, -109.2)
- moved D18 82.8 mm to (-45.8, -108.6)
- moved D20 82.8 mm to (-7.70, -108.5)
- moved D23 82.8 mm to (49.5, -108.4)
- moved D24 82.8 mm to (68.7, -108.2)
- moved D29 82.8 mm to (-97.9, -89.9)
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Routing:
- net /Column 00: track 0.00 -> 522.5 mm
- net /Column 01: track 0.00 -> 507.1 mm
- net /Column 02: track 0.00 -> 477.1 mm
- net /Column 03: track 0.00 -> 412.8 mm
- net /ROW 00: track 0.00 -> 392.0 mm, vias 0 -> 1
- net /Column 04: track 0.00 -> 389.8 mm
- net /Column 05: track 0.00 -> 365.9 mm
- net /ROW 01: track 0.00 -> 355.3 mm, vias 0 -> 1
- net /Column 06: track 0.00 -> 345.4 mm
- net /Column 07: track 0.00 -> 317.8 mm
- net /ROW 02: track 0.00 -> 299.6 mm, vias 0 -> 1
- net /Column 08: track 0.00 -> 291.6 mm
- net /ROW 03: track 0.00 -> 288.9 mm, vias 0 -> 1
- net /ROW 04: track 0.00 -> 282.8 mm, vias 0 -> 1
- net /Column 09: track 0.00 -> 243.3 mm
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Other:
- board outline added: 331.1 x 109.7 mm
