File: hardware/pcb-design.kicad_sch (KiCad schematic)
At the start: 133 parts, among them SW1 SW_MEC_5G, SW10 SW_MEC_5G, SW11 SW_MEC_5G, SW12 SW_MEC_5G, SW13 SW_MEC_5G, SW14 SW_MEC_5G, SW15 SW_MEC_5G, SW16 SW_MEC_5G, SW17 SW_MEC_5G, SW18 SW_MEC_5G, SW19 SW_MEC_5G, SW2 SW_MEC_5G, SW20 SW_MEC_5G, SW21 SW_MEC_5G, SW22 SW_MEC_5G, SW23 SW_MEC_5G, SW24 SW_MEC_5G, SW25 SW_MEC_5G, SW26 SW_MEC_5G, SW27 SW_MEC_5G, SW28 SW_MEC_5G, SW29 SW_MEC_5G, SW3 SW_MEC_5G, SW30 SW_MEC_5G, SW31 SW_MEC_5G, SW32 SW_MEC_5G, SW33 SW_MEC_5G, SW34 SW_MEC_5G, SW35 SW_MEC_5G, SW36 SW_MEC_5G, SW37 SW_MEC_5G, SW38 SW_MEC_5G, SW39 SW_MEC_5G, SW4 SW_MEC_5G, SW40 SW_MEC_5G, SW41 SW_MEC_5G, SW42 SW_MEC_5G, SW43 SW_MEC_5G, SW44 SW_MEC_5G, SW45 SW_MEC_5G, SW46 SW_MEC_5G, SW47 SW_MEC_5G, SW48 SW_MEC_5G, SW49 SW_MEC_5G, SW5 SW_MEC_5G, SW50 SW_MEC_5G, SW51 SW_MEC_5G, SW52 SW_MEC_5G, SW53 SW_MEC_5G, SW54 SW_MEC_5G, SW55 SW_MEC_5G, SW56 SW_MEC_5G, SW57 SW_MEC_5G, SW58 SW_MEC_5G, SW59 SW_MEC_5G, SW6 SW_MEC_5G, SW60 SW_MEC_5G, SW61 SW_MEC_5G, SW62 SW_MEC_5G, SW63 SW_MEC_5G, SW64 SW_MEC_5G, SW65 SW_MEC_5G, SW66 SW_MEC_5G, SW7 SW_MEC_5G, SW8 SW_MEC_5G, SW9 SW_MEC_5G

Commit message: Schemantic done
Parts:
- removed D62: D, symbol Device:D
- removed SW62: SW_MEC_5G, symbol Switch:SW_MEC_5G
- added SW67: RotaryEncoder_Switch, symbol Device:RotaryEncoder_Switch
Connections:
- net Column 00: now also A1.1 (GPIO0)
- net Column 01: now also A1.2 (GPIO1)
- net Column 02: now also A1.4 (GPIO2)
- net Column 03: now also A1.5 (GPIO3)
- net Column 04: now also A1.6 (GPIO4)
- net Column 05: now also A1.7 (GPIO5)
- net Column 06: now also A1.9 (GPIO6)
- net Column 07: now also A1.10 (GPIO7)
- net Column 08: now also A1.11 (GPIO8)
- net Column 09: now also A1.12 (GPIO9)
- net Column 10: now also A1.14 (GPIO10), D47.1 (K), D48.1 (K), D49.1 (K), D50.1 (K), D51.1 (K)
- net Column 11: now also A1.15 (GPIO11), D52.1 (K), D53.1 (K), D54.1 (K), D55.1 (K), D56.1 (K)
- net Column 12: now also A1.16 (GPIO12)
- net Column 13: now also A1.17 (GPIO13)
- net ROW 00: now also A1.29 (GPIO22); no longer A1.1 (GPIO0), A1.2 (GPIO1), SW12.1 (A), SW12.2 (A), SW17.1 (A), SW17.2 (A), SW2.1 (A), SW2.2 (A), SW22.1 (A), SW22.2 (A), SW26.1 (A), SW26.2 (A), SW30.1 (A), SW30.2 (A), SW35.1 (A), SW35.2 (A), SW39.1 (A), SW39.2 (A), SW43.1 (A), SW43.2 (A), SW47.1 (A), SW47.2 (A), SW53.1 (A), SW53.2 (A), SW58.1 (A), SW58.2 (A), SW63.1 (A), SW63.2 (A), SW7.1 (A), SW7.2 (A)
- net ROW 02: now also A1.26 (GPIO20), SW31.1 (A), SW31.2 (A), SW54.1 (A), SW54.2 (A); no longer A1.4 (GPIO2)
- net ROW 03: now also A1.25 (GPIO19); no longer A1.5 (GPIO3)
- net ROW 04: now also A1.24 (GPIO18); no longer A1.6 (GPIO4)
- net A Encoder: now reaches A1.19 (GPIO14)
- net A Encoder: now also SW67.A
- net B Encoder: now reaches A1.20 (GPIO15)
- net B Encoder: now also SW67.B
- net S1 Encoder: now reaches A1.21 (GPIO16)
- net S1 Encoder: now also SW67.S1
- net ROW 01: now reaches A1.27 (GPIO21)
- net ROW 01: now also SW12.1 (A), SW12.2 (A), SW17.1 (A), SW17.2 (A), SW2.1 (A), SW2.2 (A), SW22.1 (A), SW22.2 (A), SW26.1 (A), SW26.2 (A), SW30.1 (A), SW30.2 (A), SW35.1 (A), SW35.2 (A), SW39.1 (A), SW39.2 (A), SW43.1 (A), SW43.2 (A), SW47.1 (A), SW47.2 (A), SW53.1 (A), SW53.2 (A), SW58.1 (A), SW58.2 (A), SW63.1 (A), SW63.2 (A), SW7.1 (A), SW7.2 (A)
- new net GND: SW67.C, SW67.S2
- no-connect marks 0 -> 12
Other:
- moved on the sheet: D1, D10, D11, D12, D13, D14, D15, D16, D17, D18, D19, D2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

Commit message: Done with pcb almost
Parts:
- removed D66: D, symbol Device:D
- removed SW1, SW10, SW11, SW12, SW13, SW14, SW15, SW16, SW17, SW18, SW19, SW2, SW20, SW21, SW22, SW23, SW24, SW25, SW26, SW27, SW28, SW29, SW3, SW30, SW31, SW32, SW33, SW34, SW35, SW36, SW37, SW38, SW39, SW4, SW40, SW41, SW42, SW43, SW44, SW45, SW46, SW47, SW48, SW49, SW5, SW50, SW51, SW52, SW53, SW54, SW55, SW56, SW57, SW58, SW59, SW6, SW60, SW61, SW63, SW64, SW65, SW66, SW7, SW8, SW9: SW_MEC_5G, symbol Switch:SW_MEC_5G
- removed SW67: RotaryEncoder_Switch, symbol Device:RotaryEncoder_Switch
- added D62: D, Diode_THT:D_DO-35_SOD27_P10.16mm_Horizontal, symbol Device:D
- added MX1, MX10, MX11, MX12, MX13, MX14, MX16, MX17, MX18, MX19, MX2, MX20, MX21, MX22, MX23, MX24, MX25, MX26, MX27, MX3, MX30, MX31, MX32, MX33, MX34, MX35, MX36, MX37, MX38, MX39, MX4, MX40, MX41, MX42, MX43, MX44, MX45, MX46, MX47, MX48, MX49, MX5, MX50, MX51, MX52, MX53, MX55, MX57, MX6, MX62, MX63, MX66, MX67, MX68, MX7, MX8, MX9: MX_SW_solder, PCM_marbastlib-mx:SW_MX_1u, symbol PCM_marbastlib-mx:MX_SW_solder
- added MX15, MX28: MX_SW_solder, PCM_marbastlib-mx:SW_MX_1.5u, symbol PCM_marbastlib-mx:MX_SW_solder
- added MX29: MX_SW_solder, PCM_marbastlib-mx:SW_MX_1.75u, symbol PCM_marbastlib-mx:MX_SW_solder
- added MX54, MX56, MX58, MX59, MX60: MX_SW_solder, PCM_marbastlib-mx:SW_MX_1.25u, symbol PCM_marbastlib-mx:MX_SW_solder
- added S1: MX_stab, PCM_marbastlib-mx:STAB_MX_P_2u, symbol PCM_marbastlib-mx:MX_stab
- added S2, S3, S4: MX_stab, PCM_marbastlib-mx:STAB_MX_P_2.25u, symbol PCM_marbastlib-mx:MX_stab
- added S5: MX_stab, PCM_marbastlib-mx:STAB_MX_P_6.25u, symbol PCM_marbastlib-mx:MX_stab
- added SW62: RotaryEncoder_Switch, Rotary_Encoder:RotaryEncoder_Alps_EC11E-Switch_Vertical_H20mm, symbol Device:RotaryEncoder_Switch
- D1, D10, D11, D12, D13, D14, D15, D16, D17, D18, D19, D2, D20, D21, D22, D23, D24, D25, D26, D27, D28, D29, D3, D30, D31, D32, D33, D34, D35, D36, D37, D38, D39, D4, D40, D41, D42, D43, D44, D45, D46, D47, D48, D49, D5, D50, D51, D52, D53, D54, D55, D56, D57, D58, D59, D6, D60, D61, D63, D64, D65, D7, D8, D9: footprint (none) -> Diode_THT:D_DO-35_SOD27_P10.16mm_Horizontal
Connections:
- net A Encoder: now also A1.22 (GPIO17), SW62.A; no longer A1.19 (GPIO14)
- net B Encoder: now also A1.21 (GPIO16), SW62.B; no longer A1.20 (GPIO15)
- net Column 00: now also MX1.1, MX15.1, MX29.1, MX42.1, MX54.1; no longer D1.1 (K), D2.1 (K), D3.1 (K), D4.1 (K), D5.1 (K)
- net Column 01: now also MX16.1, MX2.1, MX30.1, MX43.1, MX55.1; no longer D10.1 (K), D6.1 (K), D7.1 (K), D8.1 (K), D9.1 (K)
- net Column 02: now also MX17.1, MX3.1, MX31.1, MX44.1, MX56.1; no longer D11.1 (K), D12.1 (K), D13.1 (K), D14.1 (K), D15.1 (K)
- net Column 03: now also MX18.1, MX32.1, MX4.1, MX45.1, MX57.1; no longer D16.1 (K), D17.1 (K), D18.1 (K), D19.1 (K), D20.1 (K)
- net Column 04: now also MX19.1, MX33.1, MX46.1, MX5.1, MX58.1; no longer D21.1 (K), D22.1 (K), D23.1 (K), D24.1 (K)
- net Column 05: now also MX20.1, MX34.1, MX47.1, MX59.1, MX6.1; no longer D25.1 (K), D26.1 (K), D27.1 (K), D28.1 (K)
- net Column 06: now also MX21.1, MX35.1, MX48.1, MX60.1, MX7.1; no longer D29.1 (K), D30.1 (K), D31.1 (K), D32.1 (K), D33.1 (K)
- net Column 07: now also MX22.1, MX36.1, MX49.1, MX66.1, MX8.1; no longer D34.1 (K), D35.1 (K), D36.1 (K), D37.1 (K)
- net Column 08: now also MX23.1, MX37.1, MX50.1, MX67.1, MX9.1; no longer D38.1 (K), D39.1 (K), D40.1 (K), D41.1 (K)
- net Column 09: now also MX10.1, MX24.1, MX38.1, MX51.1, MX68.1; no longer D42.1 (K), D43.1 (K), D44.1 (K), D45.1 (K), D46.1 (K)
- net Column 10: now also MX11.1, MX25.1, MX39.1, MX52.1; no longer D47.1 (K), D48.1 (K), D49.1 (K), D50.1 (K), D51.1 (K)
- net Column 11: now also MX12.1, MX26.1, MX40.1, MX53.1; no longer D52.1 (K), D53.1 (K), D54.1 (K), D55.1 (K), D56.1 (K)
- net Column 12: now also MX13.1, MX27.1, MX62.1; no longer D57.1 (K), D58.1 (K), D59.1 (K), D60.1 (K), D61.1 (K)
- net Column 13: now also MX14.1, MX28.1, MX41.1, MX63.1; no longer D63.1 (K), D64.1 (K), D65.1 (K)
- net GND: now also A1.13 (GND), A1.18 (GND), A1.23 (GND), A1.28 (GND), A1.3 (GND), A1.38 (GND), A1.8 (GND), SW62.C, SW62.S2
- net ROW 00: now also D54.1 (K), D55.1 (K), D56.1 (K), D57.1 (K), D58.1 (K), D59.1 (K), D60.1 (K), D61.1 (K), D64.1 (K), D65.1 (K)
- net ROW 01: now also D42.1 (K), D43.1 (K), D44.1 (K), D45.1 (K), D46.1 (K), D47.1 (K), D48.1 (K), D49.1 (K), D50.1 (K), D51.1 (K), D52.1 (K), D53.1 (K), D63.1 (K), D62.1 (K)
- net ROW 02: now also D29.1 (K), D30.1 (K), D31.1 (K), D32.1 (K), D33.1 (K), D34.1 (K), D35.1 (K), D36.1 (K), D37.1 (K), D38.1 (K), D39.1 (K), D40.1 (K), D41.1 (K)
- net ROW 03: now also D15.1 (K), D16.1 (K), D17.1 (K), D18.1 (K), D19.1 (K), D20.1 (K), D21.1 (K), D22.1 (K), D23.1 (K), D24.1 (K), D25.1 (K), D26.1 (K), D27.1 (K), D28.1 (K)
- net ROW 04: now also D1.1 (K), D10.1 (K), D11.1 (K), D12.1 (K), D13.1 (K), D14.1 (K), D2.1 (K), D3.1 (K), D4.1 (K), D5.1 (K), D6.1 (K), D7.1 (K), D8.1 (K), D9.1 (K)
- net S1 Encoder: now also A1.20 (GPIO15), SW62.S1; no longer A1.21 (GPIO16)
- net at D48.2 (A): now also MX48.2
- net at D6.2 (A): now also MX6.2
- net at D34.2 (A): now also MX34.2
- net at D59.2 (A): now also MX59.2
- net at D27.2 (A): now also MX27.2
- net at D24.2 (A): now also MX24.2
- net at D14.2 (A): now also MX14.2
- net at D12.2 (A): now also MX12.2
- net at D20.2 (A): now also MX20.2
- net at D44.2 (A): now also MX44.2
- net at D51.2 (A): now also MX51.2
- net at D13.2 (A): now also MX13.2
- net at D33.2 (A): now also MX33.2
- net at D61.2 (A): now also MX66.2
- net at D7.2 (A): now also MX7.2
- net at D63.2 (A): now also MX63.2
- net at D53.2 (A): now also MX53.2
- net at D8.2 (A): now also MX8.2
- net at D47.2 (A): now also MX47.2
- net at D9.2 (A): now also MX9.2
- net at D52.2 (A): now also MX52.2
- net at D17.2 (A): now also MX17.2
- net at D58.2 (A): now also MX58.2
- net at D46.2 (A): now also MX46.2
- net at D57.2 (A): now also MX57.2
- net at D10.2 (A): now also MX10.2
- net at D42.2 (A): now also MX42.2
- net at D31.2 (A): now also MX31.2
- net at D45.2 (A): now also MX45.2
- net at D54.2 (A): now also MX54.2
- net at D36.2 (A): now also MX36.2
- net at D50.2 (A): now also MX50.2
- net at D19.2 (A): now also MX19.2
- net at D16.2 (A): now also MX16.2
- net at D22.2 (A): now also MX22.2
- net at D30.2 (A): now also MX30.2
- net at D3.2 (A): now also MX3.2
- net at D35.2 (A): now also MX35.2
- net at D2.2 (A): now also MX2.2
- net at D18.2 (A): now also MX18.2
- net at D60.2 (A): now also MX60.2
- net at D5.2 (A): now also MX5.2
- net at D43.2 (A): now also MX43.2
- net at D26.2 (A): now also MX26.2
- net at D37.2 (A): now also MX37.2
- net at D65.2 (A): now also MX68.2
- net at D23.2 (A): now also MX23.2
- net at D21.2 (A): now also MX21.2
- net at D56.2 (A): now also MX56.2
- net at D1.2 (A): now also MX1.2
- net at D39.2 (A): now also MX39.2
- net at D49.2 (A): now also MX49.2
- net at D15.2 (A): now also MX15.2
- net at D32.2 (A): now also MX32.2
- net at D40.2 (A): now also MX40.2
- net at D11.2 (A): now also MX11.2
- net at D41.2 (A): now also MX41.2
- net at D38.2 (A): now also MX38.2
- net at D29.2 (A): now also MX29.2
- net at D55.2 (A): now also MX55.2
- net at D4.2 (A): now also MX4.2
- net at D64.2 (A): now also MX67.2
- net at D25.2 (A): now also MX25.2
- net at D28.2 (A): now also MX28.2
- new net: D62.2 (A), MX62.2
- no-connect marks 12 -> 11

Commit message: Routing done
Parts:
- removed A1: RaspberryPi_Pico, Module:RaspberryPi_Pico_Common_Unspecified, symbol MCU_Module:RaspberryPi_Pico
- removed SW62: RotaryEncoder_Switch, Rotary_Encoder:RotaryEncoder_Alps_EC11E-Switch_Vertical_H20mm, symbol Device:RotaryEncoder_Switch
- added U1: RP2040-Matrix, PCM_marbastlib-xp-promicroish:RP2040-Matrix_AC, symbol PCM_marbastlib-promicroish:RP2040-Matrix
Connections:
- net Column 00: now also U1.10 (P0)
- net Column 01: now also U1.11 (P1)
- net Column 02: now also U1.12 (P2)
- net Column 03: now also U1.13 (P3)
- net Column 04: now also U1.14 (P4)
- net Column 05: now also U1.15 (P5)
- net Column 06: now also U1.16 (P6)
- net Column 07: now also U1.17 (P7)
- net Column 08: now also U1.18 (P8)
- net Column 09: now also U1.23 (P9)
- net Column 10: now also U1.19 (P13)
- net Column 11: now also U1.20 (P12)
- net Column 12: now also U1.21 (P11)
- net Column 13: now also U1.22 (P10)
- net ROW 00: now also U1.9 (P14)
- net ROW 01: now also U1.8 (P15)
- net ROW 02: now also U1.7 (P26)
- net ROW 03: now also U1.6 (P27)
- net ROW 04: now also U1.5 (P28)
- no-connect marks 11 -> 4
