File: hardware/kicad/pcb-design.kicad_pcb (KiCad board)
At the start: 2 copper layers, 331.1 x 109.7 mm, 136 parts, among them U1 RP2040-Matrix

Commit message: key65 done
Parts:
- added H1: MountingHole, MountingHole:MountingHole_2.2mm_M2, F.Cu at (1.54, -142.4)
- added H2: MountingHole, MountingHole:MountingHole_2.2mm_M2, F.Cu at (35.6, -52.9)
- added H3: MountingHole, MountingHole:MountingHole_2.2mm_M2, F.Cu at (13.4, -56.7)
- added H4: MountingHole, MountingHole:MountingHole_2.2mm_M2, F.Cu at (-127.8, -43.5)
- added H5: MountingHole, MountingHole:MountingHole_2.2mm_M2, F.Cu at (171.4, -107.8)
- added H6: MountingHole, MountingHole:MountingHole_2.2mm_M2, F.Cu at (-131.9, -142.4)
