File: hardware/kicad/pcb-design.kicad_sch (KiCad schematic)
At the start: 136 parts, among them U1 RP2040-Matrix

Commit message: key65 done
Parts:
- added H1, H2, H3, H4, H5, H6: MountingHole, MountingHole:MountingHole_2.2mm_M2, symbol Mechanical:MountingHole
